Commit message: changed table to regular

File: models/table/table.urdf (robot description, URDF)
Before this commit: robot table.urdf, 4 links, 3 joints
Links:
- removed link guard
- removed link left_guard
- removed link right_guard
Joints:
- removed joint guard_to_surface
- removed joint left_guard_to_surface
- removed joint right_guard_to_surface
